Commit message: Añadiendo movidas del ouster

File: eufs_racecar/robots/eufs/robot.urdf.xacro (robot description, xacro)
@@ -46,7 +46,12 @@
         <origin xyz="0.0 0.0 0.4" rpy="0 0 0"/>
     </xacro:sensor_gps>
+    <!--
     <xacro:VLP-16R parent="base_footprint" name="velodyne" topic="/velodyne_points" hz="10" active="$(arg simulate_perception)">
         <origin xyz="-0.15 0.0 0.79" rpy="0 ${1*M_PI/180.0} 0"/>
     </xacro:VLP-16R>
+    -->
+    <xacro:OS1-32 parent="base_footprint" name="os1_sensor">
+        <origin xyz="-0.15 0.0 0.79" rpy="0 ${1*M_PI/180.0} 0"/>
+    </xacro:OS1-32>
     <xacro:zed_camera parent="base_footprint" prefix="zed" active="$(arg simulate_perception)">
         <origin xyz="-0.08 0.0 0.76" rpy="0 0 0"/>

File: eufs_sensors/urdf/os1-32.urdf.xacro (robot description, xacro)
@@ -1,6 +1,6 @@
 <?xml version="1.0"?>
-<robot xmlns:xacro="http://www.ros.org/wiki/xacro" name="OS1-64">
+<robot xmlns:xacro="http://www.ros.org/wiki/xacro" name="OS1-32">
   <xacro:property name="M_PI" value="3.1415926535897931" />
-  <xacro:macro name="OS1-64" params="*origin parent:=base_link name:=os1_sensor topic_points:=/os1_cloud_node/points topic_imu:=/os1_cloud_node/imu hz:=10 lasers:=64 samples:=512 min_range:=0.9 max_range:=75.0 noise:=0.008 min_angle:=-${M_PI} max_angle:=${M_PI} lidar_link:=os1_lidar imu_link:=os1_imu vfov_min:=-.26 vfov_max:=.26">
+  <xacro:macro name="OS1-32" params="*origin parent:=base_footprint name:=os1_sensor topic_points:=/ouster/points topic_imu:=/ouster/imu hz:=10 lasers:=64 samples:=512 min_range:=0.9 max_range:=75.0 noise:=0.008 min_angle:=-${M_PI} max_angle:=${M_PI} lidar_link:=os1_lidar imu_link:=os1_imu vfov_min:=-.26 vfov_max:=.26">
     <joint name="${name}_mount_joint" type="fixed">
       <xacro:insert_block name="origin" />
@@ -24,5 +24,5 @@
          <origin xyz="0 0 0.0" rpy="0 0 1.5707" />
          <geometry>
-	         <mesh filename="package://ouster_description/meshes/os1_64.dae" />
+           <mesh filename="file://$(find eufs_sensors)/meshes/os1_32.dae" />
            <!-- <cylinder length="0.073" radius="0.04" /> -->
          </geometry>
@@ -45,5 +45,5 @@
     <!-- Gazebo requires the ouster_gazebo_plugins package -->
     <gazebo reference="${name}">
-        <sensor type="ray" name="${name}-OS1-64">
+        <sensor type="ray" name="${name}-OS1-32">
           <pose>0 0 0 0 0 0</pose>
           <visualize>false</visualize>

Commit message: Editando archivos para que funcione la publicacion de mensajes

File: eufs_racecar/robots/eufs/robot.urdf.xacro (robot description, xacro)
@@ -51,5 +51,5 @@
     </xacro:VLP-16R>
     -->
-    <xacro:OS1-32 parent="base_footprint" name="os1_sensor">
+    <xacro:OS1-32 parent="base_footprint" name="os1_sensor" active="$(arg simulate_perception)">
         <origin xyz="-0.15 0.0 0.79" rpy="0 ${1*M_PI/180.0} 0"/>
     </xacro:OS1-32>

File: eufs_sensors/urdf/os1-32.urdf.xacro (robot description, xacro)
@@ -2,5 +2,5 @@
 <robot xmlns:xacro="http://www.ros.org/wiki/xacro" name="OS1-32">
   <xacro:property name="M_PI" value="3.1415926535897931" />
-  <xacro:macro name="OS1-32" params="*origin parent:=base_footprint name:=os1_sensor topic_points:=/ouster/points topic_imu:=/ouster/imu hz:=10 lasers:=64 samples:=512 min_range:=0.9 max_range:=75.0 noise:=0.008 min_angle:=-${M_PI} max_angle:=${M_PI} lidar_link:=os1_lidar imu_link:=os1_imu vfov_min:=-.26 vfov_max:=.26">
+  <xacro:macro name="OS1-32" params="*origin parent:=base_footprint name:=os1_sensor active topic_points:=/ouster/points topic_imu:=/ouster/imu hz:=10 lasers:=64 samples:=512 min_range:=0.9 max_range:=75.0 noise:=0.008 min_angle:=-${M_PI} max_angle:=${M_PI} lidar_link:=os1_lidar imu_link:=os1_imu vfov_min:=-.26 vfov_max:=.26">
     <joint name="${name}_mount_joint" type="fixed">
       <xacro:insert_block name="origin" />
