Commit message: ouster trampeado pero funcionando (sin IMU)

File: eufs_sensors/urdf/os1-32.urdf.xacro (robot description, xacro)
@@ -2,5 +2,5 @@
 <robot xmlns:xacro="http://www.ros.org/wiki/xacro" name="OS1-32">
   <xacro:property name="M_PI" value="3.1415926535897931" />
-  <xacro:macro name="OS1-32" params="*origin parent:=base_footprint name:=os1_sensor active topic_points:=/ouster/points topic_imu:=/ouster/imu hz:=10 lasers:=64 samples:=512 min_range:=0.9 max_range:=75.0 noise:=0.008 min_angle:=-${M_PI} max_angle:=${M_PI} lidar_link:=os1_lidar imu_link:=os1_imu vfov_min:=-.26 vfov_max:=.26">
+  <xacro:macro name="OS1-32" params="*origin parent:=base_footprint name:=os1_sensor active topic_points:=/ouster/points topic_imu:=/ouster/imu hz:=10 lasers:=32 samples:=512 min_range:=0.9 max_range:=75.0 noise:=0.008 min_angle:=-${M_PI} max_angle:=${M_PI} lidar_link:=os1_lidar imu_link:=os1_imu vfov_min:=-.26 vfov_max:=.26">
     <joint name="${name}_mount_joint" type="fixed">
       <xacro:insert_block name="origin" />
@@ -63,6 +63,6 @@
                 <samples>${lasers}</samples>
                 <resolution>1.0</resolution>
-                <min_angle>-${15.0*M_PI/180.0}</min_angle>
-                <max_angle> ${15.0*M_PI/180.0}</max_angle>
+                <min_angle>${vfov_min}</min_angle>
+                <max_angle>${vfov_max}</max_angle>
               </vertical>
             </scan>
@@ -80,5 +80,5 @@
           <plugin name="gazebo_ros_laser_controller" filename="libgazebo_ros_ray_sensor.so">
             <ros>
-              <remapping>~/out:=${topic}</remapping>
+              <remapping>~/out:=${topic_points}</remapping>
             </ros>
             <frame_name>${name}</frame_name>
