Commit message: cambiar transformadas camara

File: eufs_sensors/urdf/zed.urdf.xacro (robot description, xacro)
@@ -50,5 +50,5 @@
       <parent link="${prefix}_camera_center"/>
       <child link="${prefix}_depth_camera_frame"/>
-      <origin xyz="0 0.06 0" rpy="0 0 0" />
+      <origin xyz="0 0.06 0" rpy="-1.57 0 -1.57" />
     </joint>
     <!-- Simulate raw perception sensors only if we're not using the abstracted perception simulation -->
