Commit message: arreglar posicion ruedas y ocultar camara lidar

File: eufs_racecar/robots/ads-dv/robot.urdf.xacro (robot description, xacro)
@@ -31,5 +31,5 @@
     <xacro:eufs_base chassis_mesh="file://$(find eufs_racecar)/meshes/ads-dv.dae"/>
     <!-- Wheels -->
-    <xacro:wheels chassis_width="0.98" wheelbase="1.530" />
+    <xacro:wheels chassis_width="1.28" wheelbase="1.4" />
     <!-- *********************************************** -->
     <!--                 MAIN SENSORS                    -->
@@ -40,4 +40,5 @@
     LIDAR: 1.700 0.0 -0.150
     STEREO CAM: -0.110 0.0 0.800 -->
+    <!--
     <xacro:sensor_imu parent="base_footprint" prefix="imu">
         <origin xyz="0.0 0.0 0.0" rpy="0 0 0"/>
@@ -52,3 +53,4 @@
 	<origin xyz="0.12 0.0 0.76" rpy="0 ${10.15*M_PI/180.0} 0"/>
     </xacro:zed_camera>
+    -->
 </robot>

File: eufs_racecar/urdf/wheels.urdf.xacro (robot description, xacro)
@@ -32,5 +32,5 @@
         </inertial>
         <visual>
-          <origin xyz="0 0 0" rpy="${degrees_90} 0 0"/>
+          <origin xyz="-0.4 0 -0.1" rpy="${degrees_90} 0 0"/>
           <geometry>
             <mesh filename="file://$(find eufs_racecar)/meshes/wheel_${lr_prefix}.dae"/>

Commit message: deberes de la placa

File: eufs_racecar/robots/ads-dv/robot.urdf.xacro (robot description, xacro)
@@ -32,23 +32,20 @@
     <!-- Wheels -->
     <xacro:wheels chassis_width="0.98" wheelbase="1.530" />
-    <!-- *********************************************** -->
-    <!--                 MAIN SENSORS                    -->
-    <!-- *********************************************** -->
-    <!--     LOCATIONS: (XYZ)
-    IMU: 0.0 0.0 0.170
-    GPS: -0.110 0.0 0.9
-    LIDAR: 1.700 0.0 -0.150
-    STEREO CAM: -0.110 0.0 0.800 -->
-    <xacro:sensor_imu parent="base_footprint" prefix="imu">
-        <origin xyz="0.0 0.0 0.0" rpy="0 0 0"/>
+    <!-- Placa -->
+    <xacro:plate prefix="plate" parent="base_footprint">
+        <origin xyz="0 0 0.05" rpy="0 0 0"/>
+    </xacro:plate>
+    <!-- Sensores -->
+    <xacro:sensor_imu parent="plate_plate" prefix="imu">
+        <origin xyz="1 1 1" rpy="0 0 0"/>
     </xacro:sensor_imu>
-    <xacro:sensor_gps parent="base_footprint" prefix="gps">
+    <xacro:sensor_gps parent="plate_plate" prefix="gps">
         <origin xyz="0.0 0.0 0.4" rpy="0 0 0"/>
     </xacro:sensor_gps>
-    <xacro:VLP-16R parent="base_footprint" name="velodyne" topic="/velodyne_points" hz="10" samples="800" active="$(arg simulate_perception)">
-	<origin xyz="0.59 0.0 0.51" rpy="0 ${10*M_PI/180.0} 0"/>
+    <xacro:VLP-16R parent="plate_plate" name="velodyne" topic="/velodyne_points" hz="10" samples="800" active="$(arg simulate_perception)">
+        <origin xyz="0.59 0.0 0.51" rpy="0 ${10*PI/180.0} 0"/>
     </xacro:VLP-16R>
-    <xacro:zed_camera parent="base_footprint" prefix="zed" active="$(arg simulate_perception)">
-	<origin xyz="0.12 0.0 0.76" rpy="0 ${10.15*M_PI/180.0} 0"/>
+    <xacro:zed_camera parent="plate_plate" prefix="zed" active="$(arg simulate_perception)">
+        <origin xyz="0.12 0.0 0.76" rpy="0 ${10.15*PI/180.0} 0"/>
     </xacro:zed_camera>
 </robot>

File: eufs_sensors/urdf/all_sensors.urdf.xacro (robot description, xacro)
@@ -10,3 +10,5 @@
   <!-- ZED Stereo camera -->
   <xacro:include filename="$(find eufs_sensors)/urdf/zed.urdf.xacro"/>
+    <!-- Plate -->
+  <xacro:include filename="$(find eufs_sensors)/urdf/plate.urdf.xacro"/>
 </robot>

Commit message: Placa de sensores añadida

File: eufs_racecar/robots/ads-dv/robot.urdf.xacro (robot description, xacro)
@@ -34,18 +34,18 @@
     <!-- Placa -->
     <xacro:plate prefix="plate" parent="base_footprint">
-        <origin xyz="0 0 0.05" rpy="0 0 0"/>
+        <origin xyz="0.5 0 0.2" rpy="0 0 0"/>
     </xacro:plate>
     <!-- Sensores -->
     <xacro:sensor_imu parent="plate_plate" prefix="imu">
-        <origin xyz="1 1 1" rpy="0 0 0"/>
+        <origin xyz="0 0 0" rpy="0 0 0"/>
     </xacro:sensor_imu>
     <xacro:sensor_gps parent="plate_plate" prefix="gps">
-        <origin xyz="0.0 0.0 0.4" rpy="0 0 0"/>
+        <origin xyz="0 0 0" rpy="0 0 0"/>
     </xacro:sensor_gps>
-    <xacro:VLP-16R parent="plate_plate" name="velodyne" topic="/velodyne_points" hz="10" samples="800" active="$(arg simulate_perception)">
-        <origin xyz="0.59 0.0 0.51" rpy="0 ${10*PI/180.0} 0"/>
-    </xacro:VLP-16R>
+    <xacro:OS1-32 parent="plate_plate" name="os1_sensor" active="$(arg simulate_perception)">
+        <origin xyz="0.1 0.0 0.15" rpy="0 0 0"/>
+    </xacro:OS1-32>
     <xacro:zed_camera parent="plate_plate" prefix="zed" active="$(arg simulate_perception)">
-        <origin xyz="0.12 0.0 0.76" rpy="0 ${10.15*PI/180.0} 0"/>
+        <origin xyz="-0.03 0.0 0.23" rpy="0 ${10.15*PI/180.0} 0"/>
     </xacro:zed_camera>
 </robot>

File: eufs_sensors/urdf/all_sensors.urdf.xacro (robot description, xacro)
@@ -2,15 +2,15 @@
 <robot name="all_sensors" xmlns:xacro="http://www.ros.org/wiki/xacro">
   <!-- This file unifies all sensors that can be used on simulation, defined as xacro:macros -->
+  <!-- Plate -->
+  <xacro:include filename="$(find eufs_sensors)/urdf/plate.urdf.xacro"/>
   <!-- GPS -->
   <xacro:include filename="$(find eufs_sensors)/urdf/gps.urdf.xacro"/>
   <!-- Velodyne VLP-16R -->
-  <xacro:include filename="$(find eufs_sensors)/urdf/VLP-16R.urdf.xacro"/>
+  <!-- <xacro:include filename="$(find eufs_sensors)/urdf/VLP-16R.urdf.xacro"/> -->
   <!-- Ouster OS1-32 -->
-  <xacro:include filename="$(find eufs_sensors)/urdf/os1-32.urdf.xacro"/>
+  <xacro:include filename="$(find eufs_sensors)/urdf/os1-32.urdf.xacro" parent="plate_link"/>
   <!-- Imu -->
   <xacro:include filename="$(find eufs_sensors)/urdf/imu.urdf.xacro"/>
   <!-- ZED Stereo camera -->
-  <xacro:include filename="$(find eufs_sensors)/urdf/zed.urdf.xacro"/>
-    <!-- Plate -->
-  <xacro:include filename="$(find eufs_sensors)/urdf/plate.urdf.xacro"/>
+  <xacro:include filename="$(find eufs_sensors)/urdf/zed.urdf.xacro" parent="plate_link"/>
 </robot>

File: eufs_sensors/urdf/plate.urdf.xacro (robot description, xacro)
@@ -1,5 +1,5 @@
 <?xml version="1.0"?>
 <robot name="plate" xmlns:xacro="http://www.ros.org/wiki/xacro">
-  <xacro:macro name="plate" params="prefix parent *origin">
+  <xacro:macro name="plate" params="*origin parent:=base_footprint prefix">
     <link name="${prefix}_plate">
       <inertial>
@@ -9,5 +9,5 @@
       </inertial>
       <visual>
-        <origin xyz="0 0 0" rpy="0 0 0"/>
+        <origin xyz="-0.6 0 -0.15" rpy="0 0 0"/>
         <geometry>
           <mesh filename="file://$(find eufs_sensors)/meshes/plate.dae" scale="1 1 1"/>
@@ -23,5 +23,5 @@
     </link>
     <joint name="${prefix}_base_joint" type="fixed">
-      <axis xyz="1 0 0"/>
+      <axis xyz="0 0 0"/>
       <xacro:insert_block name="origin"/>
       <parent link="${parent}"/>
